File: keyboard-tutorial.kicad_sch (KiCad schematic)
At the start: 0 parts

Commit message: added decoupling capacitors and ISP header
Parts:
- added C1: 1u, symbol Device:C_Small
- added C2, C3: 22p, symbol Device:C_Small
- added C4, C6, C7, C8: 0.1u, symbol Device:C_Small
- added C5: 10u, symbol Device:C_Small
- added J1: AVR-ISP-6, symbol Connector:AVR-ISP-6
- added R1: 10k, symbol Device:R_Small
- added U1: ATmega32U4-A, Package_QFP:TQFP-44_10x10mm_P0.8mm, symbol MCU_Microchip_ATmega:ATmega32U4-A
- added Y1: XTAL, symbol Device:Crystal_GND24_Small
Connections:
- new net: R1.1, U1.33 (~{HWB}/PE2)
- new net: C1.1, U1.6 (UCAP)
- new net +5V: C4.1, C5.1, C6.1, C7.1, C8.1, J1.2 (VCC), U1.14 (VCC), U1.2 (UVCC), U1.24 (AVCC), U1.34 (VCC), U1.44 (AVCC)
- new net D+: U1.4 (D+)
- new net D-: U1.3 (D-)
- new net GND: C1.2, C2.2, C3.2, C4.2, C5.2, C6.2, C7.2, C8.2, J1.6 (GND), R1.2, U1.15 (GND), U1.23 (GND), U1.35 (GND), U1.43 (GND), U1.5 (UGND), Y1.2, Y1.4
- new net MISO: J1.1 (MISO), U1.11 (PB3)
- new net MOSI: J1.4 (MOSI), U1.10 (PB2)
- new net RESET: J1.5 (~{RST}), U1.13 (~{RESET})
- new net SCK: J1.3 (SCK), U1.9 (PB1)
- new net XTAL1: C2.1, U1.17 (XTAL1), Y1.1
- new net XTAL2: C3.1, U1.16 (XTAL2), Y1.3
- no-connect marks 0 -> 1
